File: hardware/peripheral/p2gpl-001.sch (EAGLE design)
At the start: 4 parts, among them J11 AUDIO_JACK_3.5MM_KIT

Commit message: Fixed polarity of 3.5mm jack.
Connections:
- net ANLG0: now also J11.TIP; no longer J11.RING
- net VCC: now also J11.RING; no longer J11.TIP
Changed lines of the file:
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@@
 </segment>
 <segment>
-<pinref part="J11" gate="G$1" pin="TIP"/>
-<wire x1="66.04" y1="96.52" x2="68.58" y2="96.52" width="0.1524" layer="91"/>
-<label x="68.58" y="96.52" size="0.8128" layer="95" xref="yes"/>
+<pinref part="J11" gate="G$1" pin="RING"/>
+<wire x1="66.04" y1="104.14" x2="68.58" y2="104.14" width="0.1524" layer="91"/>
+<label x="68.58" y="104.14" size="0.8128" layer="95" xref="yes"/>
 </segment>
 </net>
@@
 </segment>
 <segment>
-<pinref part="J11" gate="G$1" pin="RING"/>
-<wire x1="66.04" y1="104.14" x2="68.58" y2="104.14" width="0.1524" layer="91"/>
-<label x="68.58" y="104.14" size="0.8128" layer="95" xref="yes"/>
+<pinref part="J11" gate="G$1" pin="TIP"/>
+<wire x1="66.04" y1="96.52" x2="68.58" y2="96.52" width="0.1524" layer="91"/>
+<label x="68.58" y="96.52" size="0.8128" layer="95" xref="yes"/>
 </segment>
 </net>
